File: pcbs/rpi_hat/rpi_hat.sch (EAGLE design)
At the start: 13 parts, among them J2 RJ11-2L-B

Commit message: Added the dataready line
Connections:
- new net N$3: J2.5, SV1.15
- net N$1: no longer J2.5
Changed lines of the file:
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@@
 <net name="N$1" class="0">
 <segment>
-<pinref part="J2" gate="G$1" pin="5"/>
-<wire x1="101.6" y1="20.32" x2="111.76" y2="20.32" width="0.1524" layer="91"/>
-<wire x1="111.76" y1="20.32" x2="111.76" y2="22.86" width="0.1524" layer="91"/>
 <wire x1="111.76" y1="22.86" x2="111.76" y2="58.42" width="0.1524" layer="91"/>
 <wire x1="111.76" y1="58.42" x2="137.16" y2="58.42" width="0.1524" layer="91"/>
@@
 <pinref part="J2" gate="G$1" pin="6"/>
 <wire x1="101.6" y1="22.86" x2="111.76" y2="22.86" width="0.1524" layer="91"/>
-<junction x="111.76" y="22.86"/>
 <pinref part="R1" gate="G$1" pin="2"/>
 <wire x1="144.78" y1="30.48" x2="144.78" y2="58.42" width="0.1524" layer="91"/>
@@
 </segment>
 </net>
+<net name="N$3" class="0">
+<segment>
+<pinref part="J2" gate="G$1" pin="5"/>
+<wire x1="101.6" y1="20.32" x2="116.84" y2="20.32" width="0.1524" layer="91"/>
+<wire x1="116.84" y1="20.32" x2="116.84" y2="93.98" width="0.1524" layer="91"/>
+<pinref part="SV1" gate="G$1" pin="15"/>
+<wire x1="116.84" y1="93.98" x2="195.58" y2="93.98" width="0.1524" layer="91"/>
+<wire x1="195.58" y1="93.98" x2="195.58" y2="60.96" width="0.1524" layer="91"/>
+</segment>
+</net>
