File: pcbs/imu_board/imu_board.sch (EAGLE design)
At the start: 25 parts, among them J1 RJ11-2L-B, U1 LSM9DS1, U2 ADP121-AUJZ33R7

Commit message: Added the dataready line
Connections:
- new net N$3: J1.5, U1.DRDY_M
- net N$46: no longer J1.5
Changed lines of the file:
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@@
 <net name="N$46" class="0">
 <segment>
-<pinref part="J1" gate="G$1" pin="5"/>
-<wire x1="-185.42" y1="76.2" x2="-175.26" y2="76.2" width="0.1524" layer="91"/>
-<wire x1="-175.26" y1="76.2" x2="-175.26" y2="78.74" width="0.1524" layer="91"/>
 <wire x1="-175.26" y1="78.74" x2="-175.26" y2="114.3" width="0.1524" layer="91"/>
 <wire x1="-175.26" y1="114.3" x2="-152.4" y2="114.3" width="0.1524" layer="91"/>
@@
 <pinref part="J1" gate="G$1" pin="6"/>
 <wire x1="-185.42" y1="78.74" x2="-175.26" y2="78.74" width="0.1524" layer="91"/>
-<junction x="-175.26" y="78.74"/>
 <pinref part="R7" gate="G$1" pin="2"/>
 <wire x1="-144.78" y1="86.36" x2="-144.78" y2="114.3" width="0.1524" layer="91"/>
@@
 </segment>
 </net>
+<net name="N$3" class="0">
+<segment>
+<pinref part="J1" gate="G$1" pin="5"/>
+<wire x1="-185.42" y1="76.2" x2="-167.64" y2="76.2" width="0.1524" layer="91"/>
+<wire x1="-167.64" y1="76.2" x2="-167.64" y2="124.46" width="0.1524" layer="91"/>
+<wire x1="-167.64" y1="124.46" x2="-58.42" y2="124.46" width="0.1524" layer="91"/>
+<wire x1="-58.42" y1="124.46" x2="-58.42" y2="55.88" width="0.1524" layer="91"/>
+<pinref part="U1" gate="G$1" pin="DRDY_M"/>
+<wire x1="-58.42" y1="55.88" x2="15.24" y2="55.88" width="0.1524" layer="91"/>
+</segment>
+</net>

Commit message: Updated docs
Connections:
- net N$3: now also U1.INT2_A/G; no longer U1.DRDY_M
Changed lines of the file:
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@@
 <wire x1="-167.64" y1="76.2" x2="-167.64" y2="124.46" width="0.1524" layer="91"/>
 <wire x1="-167.64" y1="124.46" x2="-58.42" y2="124.46" width="0.1524" layer="91"/>
-<wire x1="-58.42" y1="124.46" x2="-58.42" y2="55.88" width="0.1524" layer="91"/>
-<pinref part="U1" gate="G$1" pin="DRDY_M"/>
-<wire x1="-58.42" y1="55.88" x2="15.24" y2="55.88" width="0.1524" layer="91"/>
+<wire x1="-58.42" y1="124.46" x2="-58.42" y2="63.5" width="0.1524" layer="91"/>
+<pinref part="U1" gate="G$1" pin="INT2_A/G"/>
+<wire x1="15.24" y1="63.5" x2="-58.42" y2="63.5" width="0.1524" layer="91"/>
 </segment>
 </net>
